File: pcb/wiproc/wiproc/batt_chrg.sch (KiCad schematic (older format))
At the start: 9 parts, among them U5 TLV70033_SOT23-5, U6 MCP73831-2-OT

Commit message: routed wiproc, created synth pcb
Parts:
- added J7: Conn_01x02, Connector_JST:JST_PH_S2B-PH-SM4-TB_1x02-1MP_P2.00mm_Horizontal, symbol Connector_Generic:Conn_01x02
- C14: renamed from C16; footprint (none) -> Capacitor_SMD:C_0603_1608Metric_Pad1.05x0.95mm_HandSolder
- C15: renamed from C17; footprint (none) -> Capacitor_SMD:C_0603_1608Metric_Pad1.05x0.95mm_HandSolder
- C16: renamed from C14; footprint (none) -> Capacitor_SMD:C_0603_1608Metric_Pad1.05x0.95mm_HandSolder
- C17: renamed from C15; footprint (none) -> Capacitor_SMD:C_0603_1608Metric_Pad1.05x0.95mm_HandSolder
- D6: footprint (none) -> LED_SMD:LED_0805_2012Metric_Pad1.15x1.40mm_HandSolder
- R17, R18: footprint (none) -> Resistor_SMD:R_0603_1608Metric_Pad1.05x0.95mm_HandSolder
Connections:
- net +BATT: now also J7.1 (Pin_1)
- net GND: now also J7.2 (Pin_2)
Other:
- moved on the sheet: C14, C15, C16, C17, D6, R17, R18, U5, U6
