File: pcb/wiproc/wiproc/mcu_atmega328p.sch (KiCad schematic (older format))
At the start: 24 parts, among them J4 Conn_02x03_Odd_Even, SW1 SW_Push, SW2 SW_Push, SW3 SW_Push, SW4 SW_Push, U1 ATmega328P-AU, Y1 Crystal

Commit message: routed wiproc, created synth pcb
Parts:
- removed U1: ATmega328P-AU, Package_QFP:TQFP-32_7x7mm_P0.8mm, symbol MCU_Microchip_ATmega:ATmega328P-AU
- added U1: ATmega328P-AU, Package_QFP:TQFP-32_7x7mm_P0.8mm, symbol atmega48p:ATmega328P-AU
- C2, C3, C4, C5: footprint (none) -> Capacitor_SMD:C_0603_1608Metric_Pad1.05x0.95mm_HandSolder
- C6, C7: value C -> 18pF; footprint (none) -> Capacitor_SMD:C_0603_1608Metric_Pad1.05x0.95mm_HandSolder
- D1, D2: footprint (none) -> LED_SMD:LED_0805_2012Metric_Pad1.15x1.40mm_HandSolder
- J4: footprint (none) -> Connector_PinHeader_2.54mm:PinHeader_2x03_P2.54mm_Vertical_SMD
- R1, R2, R3, R4, R5, R6, R7, R8, R9: footprint (none) -> Resistor_SMD:R_0603_1608Metric_Pad1.05x0.95mm_HandSolder
- SW1, SW2, SW3, SW4: footprint (none) -> Button_Switch_SMD:SW_SPST_TL3342
- Y1: value Crystal -> 16MHz; footprint (none) -> Crystal:Crystal_SMD_ECS_CSM3X-2Pin_7.6x4.1mm; PN (none) -> ABLS7M
Connections:
- net +3V3: now also U1.18 (AVCC), U1.20 (AREF), U1.4 (VCC), U1.6 (VCC)
- net ADC_IN1: now also U1.19 (ADC6)
- net ADC_IN2: now also U1.22 (ADC7)
- net GND: now also U1.21 (GND), U1.3 (GND), U1.5 (GND)
- net I2C_SCL: now also U1.28 (PC5)
- net I2C_SDA: now also U1.27 (PC4)
- net MCU_BTN1: now also U1.23 (PC0)
- net MCU_BTN2: now also U1.24 (PC1)
- net MCU_BTN3: now also U1.25 (PC2)
- net MCU_BTN4: now also U1.26 (PC3)
- net MCU_LED1: now also U1.32 (PD2)
- net MCU_LED2: now also U1.1 (PD3)
- net MCU_RST_N: now also U1.29 (~RESET~/PC6)
- net SPARE_IO_1: now also U1.2 (PD4)
- net SPARE_IO_2: now also U1.9 (PD5)
- net SPI_ATTN_N: now also U1.13 (PB1)
- net SPI_CLK: now also U1.17 (PB5)
- net SPI_MISO: now also U1.16 (PB4)
- net SPI_MOSI: now also U1.15 (PB3)
- net SPI_SS_N: now also U1.14 (PB2)
- net UART_RX: now also U1.30 (PD0)
- net UART_TX: now also U1.31 (PD1)
- net XBEE_DOUT: now also U1.10 (PD6)
- net XBEE_RST_N: now also U1.11 (PD7)
- net XTAL1_16MHZ: now also U1.7 (XTAL1/PB6)
- net XTAL2_16MHZ: now also U1.8 (XTAL2/PB7)
Changed lines of the file:
@@
 $Descr A4 11693 8268
 encoding utf-8
-Sheet 2 4
+Sheet 2 5
 Title ""
 Date ""
@@
 Comment4 ""
 $EndDescr
-$Comp
-L MCU_Microchip_ATmega:ATmega328P-AU U1
-U 1 1 5DAA3BFB
-P 3500 4400
-F 0 "U1" H 3500 3350 50  0000 C CNN
-F 1 "ATmega328P-AU" H 3500 3250 50  0000 C CNN
-F 2 "Package_QFP:TQFP-32_7x7mm_P0.8mm" H 3500 4400 50  0001 C CIN
-F 3 "http://ww1.microchip.com/downloads/en/DeviceDoc/ATmega328_P%20AVR%20MCU%20with%20picoPower%20Technology%20Data%20Sheet%2040001984A.pdf" H 3500 4400 50  0001 C CNN
-	1    3500 4400
-	1    0    0    -1
-$EndComp
 Wire Wire Line
 	4100 3500 6200 3500
@@
 U 1 1 5DAA3C04
 P 6250 6200
-F 0 "Y1" H 6250 5932 50  0000 C CNN
-F 1 "Crystal" H 6250 6023 50  0000 C CNN
-F 2 "" H 6250 6200 50  0001 C CNN
+F 0 "Y1" H 5900 6000 50  0000 C CNN
+F 1 "16MHz" H 5900 6100 50  0000 C CNN
+F 2 "Crystal:Crystal_SMD_ECS_CSM3X-2Pin_7.6x4.1mm" H 6250 6200 50  0001 C CNN
 F 3 "~" H 6250 6200 50  0001 C CNN
+F 4 "ABLS7M" H 5900 6200 50  0000 C CNN "PN"
 	1    6250 6200
 	-1   0    0    1
@@
 P 6100 6500
 F 0 "C6" H 5986 6546 50  0000 R CNN
-F 1 "C" H 5986 6455 50  0000 R CNN
-F 2 "" H 6138 6350 50  0001 C CNN
+F 1 "18pF" H 5986 6455 50  0000 R CNN
+F 2 "Capacitor_SMD:C_0603_1608Metric_Pad1.05x0.95mm_HandSolder" H 6138 6350 50  0001 C CNN
 F 3 "~" H 6100 6500 50  0001 C CNN
 	1    6100 6500
@@
 P 6400 6500
 F 0 "C7" H 6515 6546 50  0000 L CNN
-F 1 "C" H 6515 6455 50  0000 L CNN
-F 2 "" H 6438 6350 50  0001 C CNN
+F 1 "18pF" H 6515 6455 50  0000 L CNN
+F 2 "Capacitor_SMD:C_0603_1608Metric_Pad1.05x0.95mm_HandSolder" H 6438 6350 50  0001 C CNN
 F 3 "~" H 6400 6500 50  0001 C CNN
 	1    6400 6500
@@
 F 0 "J4" H 5650 2450 50  0000 C CNN
 F 1 "Conn_02x03_Odd_Even" H 6700 2750 50  0000 C CNN
-F 2 "" H 5600 2700 50  0001 C CNN
+F 2 "Connector_PinHeader_2.54mm:PinHeader_2x03_P2.54mm_Vertical_SMD" H 5600 2700 50  0001 C CNN
 F 3 "~" H 5600 2700 50  0001 C CNN
 	1    5600 2700
@@
 F 0 "C2" H 1715 2646 50  0000 L CNN
 F 1 "0.1uF" H 1715 2555 50  0000 L CNN
-F 2 "" H 1638 2450 50  0001 C CNN
+F 2 "Capacitor_SMD:C_0603_1608Metric_Pad1.05x0.95mm_HandSolder" H 1638 2450 50  0001 C CNN
 F 3 "~" H 1600 2600 50  0001 C CNN
 	1    1600 2600
@@
 F 0 "C4" H 2615 2646 50  0000 L CNN
 F 1 "0.1uF" H 2615 2555 50  0000 L CNN
-F 2 "" H 2538 2450 50  0001 C CNN
+F 2 "Capacitor_SMD:C_0603_1608Metric_Pad1.05x0.95mm_HandSolder" H 2538 2450 50  0001 C CNN
 F 3 "~" H 2500 2600 50  0001 C CNN
 	1    2500 2600
@@
 F 0 "C3" H 2165 2646 50  0000 L CNN
 F 1 "0.1uF" H 2165 2555 50  0000 L CNN
-F 2 "" H 2088 2450 50  0001 C CNN
+F 2 "Capacitor_SMD:C_0603_1608Metric_Pad1.05x0.95mm_HandSolder" H 2088 2450 50  0001 C CNN
 F 3 "~" H 2050 2600 50  0001 C CNN
 	1    2050 2600
@@
 F 0 "R5" H 5368 2346 50  0000 L CNN
 F 1 "10k" H 5368 2255 50  0000 L CNN
-F 2 "" V 5340 2290 50  0001 C CNN
+F 2 "Resistor_SMD:R_0603_1608Metric_Pad1.05x0.95mm_HandSolder" V 5340 2290 50  0001 C CNN
 F 3 "~" H 5300 2300 50  0001 C CNN
 	1    5300 2300
@@
 F 0 "R7" H 8768 4146 50  0000 L CNN
 F 1 "10k" H 8768 4055 50  0000 L CNN
-F 2 "" V 8740 4090 50  0001 C CNN
+F 2 "Resistor_SMD:R_0603_1608Metric_Pad1.05x0.95mm_HandSolder" V 8740 4090 50  0001 C CNN
 F 3 "~" H 8700 4100 50  0001 C CNN
 	1    8700 4100
@@
 F 0 "R6" H 8432 4146 50  0000 R CNN
 F 1 "10k" H 8432 4055 50  0000 R CNN
-F 2 "" V 8540 4090 50  0001 C CNN
+F 2 "Resistor_SMD:R_0603_1608Metric_Pad1.05x0.95mm_HandSolder" V 8540 4090 50  0001 C CNN
 F 3 "~" H 8500 4100 50  0001 C CNN
 	1    8500 4100
@@
 F 0 "D1" H 8643 4795 50  0000 C CNN
 F 1 "LED" H 8643 4886 50  0000 C CNN
-F 2 "" H 8650 5050 50  0001 C CNN
+F 2 "LED_SMD:LED_0805_2012Metric_Pad1.15x1.40mm_HandSolder" H 8650 5050 50  0001 C CNN
 F 3 "~" H 8650 5050 50  0001 C CNN
 	1    8650 5050
@@
 F 0 "D2" H 8643 5373 50  0000 C CNN
 F 1 "LED" H 8643 5464 50  0000 C CNN
-F 2 "" H 8650 5250 50  0001 C CNN
+F 2 "LED_SMD:LED_0805_2012Metric_Pad1.15x1.40mm_HandSolder" H 8650 5250 50  0001 C CNN
 F 3 "~" H 8650 5250 50  0001 C CNN
 	1    8650 5250
@@
 F 0 "R8" V 7345 5050 50  0000 C CNN
 F 1 "220" V 7436 5050 50  0000 C CNN
-F 2 "" V 7590 5040 50  0001 C CNN
+F 2 "Resistor_SMD:R_0603_1608Metric_Pad1.05x0.95mm_HandSolder" V 7590 5040 50  0001 C CNN
 F 3 "~" H 7550 5050 50  0001 C CNN
 	1    7550 5050
@@
 F 0 "R9" V 7663 5250 50  0000 C CNN
 F 1 "220" V 7754 5250 50  0000 C CNN
-F 2 "" V 7590 5240 50  0001 C CNN
+F 2 "Resistor_SMD:R_0603_1608Metric_Pad1.05x0.95mm_HandSolder" V 7590 5240 50  0001 C CNN
 F 3 "~" H 7550 5250 50  0001 C CNN
 	1    7550 5250
@@
 F 0 "C5" H 9265 5196 50  0000 L CNN
 F 1 "0.1uF" H 9265 5105 50  0000 L CNN
-F 2 "" H 9188 5000 50  0001 C CNN
+F 2 "Capacitor_SMD:C_0603_1608Metric_Pad1.05x0.95mm_HandSolder" H 9188 5000 50  0001 C CNN
 F 3 "~" H 9150 5150 50  0001 C CNN
 	1    9150 5150
@@
 F 0 "SW1" H 9750 2185 50  0000 C CNN
 F 1 "SW_Push" H 9750 2094 50  0000 C CNN
-F 2 "" H 9750 2100 50  0001 C CNN
+F 2 "Button_Switch_SMD:SW_SPST_TL3342" H 9750 2100 50  0001 C CNN
 F 3 "~" H 9750 2100 50  0001 C CNN
 	1    9750 1900
@@
 F 0 "SW2" H 10250 2535 50  0000 C CNN
 F 1 "SW_Push" H 10250 2444 50  0000 C CNN
-F 2 "" H 10250 2450 50  0001 C CNN
+F 2 "Button_Switch_SMD:SW_SPST_TL3342" H 10250 2450 50  0001 C CNN
 F 3 "~" H 10250 2450 50  0001 C CNN
 	1    10250 2250
@@
 F 0 "SW3" H 9800 2885 50  0000 C CNN
 F 1 "SW_Push" H 9800 2794 50  0000 C CNN
-F 2 "" H 9800 2800 50  0001 C CNN
+F 2 "Button_Switch_SMD:SW_SPST_TL3342" H 9800 2800 50  0001 C CNN
 F 3 "~" H 9800 2800 50  0001 C CNN
 	1    9800 2600
@@
 F 0 "SW4" H 10300 3235 50  0000 C CNN
 F 1 "SW_Push" H 10300 3144 50  0000 C CNN
-F 2 "" H 10300 3150 50  0001 C CNN
+F 2 "Button_Switch_SMD:SW_SPST_TL3342" H 10300 3150 50  0001 C CNN
 F 3 "~" H 10300 3150 50  0001 C CNN
 	1    10300 2950
@@
 F 0 "R4" H 9132 1596 50  0000 R CNN
 F 1 "10k" H 9132 1505 50  0000 R CNN
-F 2 "" V 9240 1540 50  0001 C CNN
+F 2 "Resistor_SMD:R_0603_1608Metric_Pad1.05x0.95mm_HandSolder" V 9240 1540 50  0001 C CNN
 F 3 "~" H 9200 1550 50  0001 C CNN
 	1    9200 1550
@@
 F 0 "R3" H 8832 1596 50  0000 R CNN
 F 1 "10k" H 8832 1505 50  0000 R CNN
-F 2 "" V 8940 1540 50  0001 C CNN
+F 2 "Resistor_SMD:R_0603_1608Metric_Pad1.05x0.95mm_HandSolder" V 8940 1540 50  0001 C CNN
 F 3 "~" H 8900 1550 50  0001 C CNN
 	1    8900 1550
@@
 F 0 "R2" H 8532 1596 50  0000 R CNN
 F 1 "10k" H 8532 1505 50  0000 R CNN
-F 2 "" V 8640 1540 50  0001 C CNN
+F 2 "Resistor_SMD:R_0603_1608Metric_Pad1.05x0.95mm_HandSolder" V 8640 1540 50  0001 C CNN
 F 3 "~" H 8600 1550 50  0001 C CNN
 	1    8600 1550
@@
 F 0 "R1" H 8232 1596 50  0000 R CNN
 F 1 "10k" H 8232 1505 50  0000 R CNN
-F 2 "" V 8340 1540 50  0001 C CNN
+F 2 "Resistor_SMD:R_0603_1608Metric_Pad1.05x0.95mm_HandSolder" V 8340 1540 50  0001 C CNN
 F 3 "~" H 8300 1550 50  0001 C CNN
 	1    8300 1550
@@
 I2C_SCL
 NoConn ~ 4100 3200
+$Comp
+L atmega48p:ATmega328P-AU U1
+U 1 1 5DB3C0E0
+P 3500 4400
+F 0 "U1" H 3500 4500 50  0000 C CNN
+F 1 "ATmega328P-AU" H 3450 4350 50  0000 C CNN
+F 2 "Package_QFP:TQFP-32_7x7mm_P0.8mm" H 3500 4400 50  0001 C CIN
+F 3 "http://ww1.microchip.com/downloads/en/DeviceDoc/ATmega328_P%20AVR%20MCU%20with%20picoPower%20Technology%20Data%20Sheet%2040001984A.pdf" H 3500 4400 50  0001 C CNN
+	1    3500 4400
+	1    0    0    -1
+$EndComp
 $EndSCHEMATC
