File: pcb/wiproc/wiproc/usb_uart.sch (KiCad schematic (older format))
At the start: 21 parts, among them J5 Conn_01x02_Male, J6 USB_B_Micro, U2 FODM8071, U3 74LVC1G97, U4 FT231XS

Commit message: routed wiproc, created synth pcb
Parts:
- removed U2: FODM8071, Package_DIP:DIP-6_W7.62mm, symbol Isolator:4N35
- added U2: FODM8071, Package_SO:SO-5_4.4x3.6mm_P1.27mm, symbol wiproc-rescue:FODM8071-fodm8071
- C10, C11, C12, C13, C8, C9: footprint (none) -> Capacitor_SMD:C_0603_1608Metric_Pad1.05x0.95mm_HandSolder
- D3: value D -> 1N4148WS; footprint (none) -> Diode_SMD:D_SOD-323_HandSoldering
- D4, D5: footprint (none) -> LED_SMD:LED_0805_2012Metric_Pad1.15x1.40mm_HandSolder
- J5: footprint (none) -> Connector_PinHeader_2.54mm:PinHeader_1x02_P2.54mm_Vertical
- J6: footprint (none) -> Connector_USB:USB_Micro-B_Molex_47346-0001
- R10, R11, R12, R13, R14, R15, R16: footprint (none) -> Resistor_SMD:R_0603_1608Metric_Pad1.05x0.95mm_HandSolder
- U3: footprint (none) -> Package_TO_SOT_SMD:SOT-23-6
Connections:
- net +3V3: now also U2.6
- net GND: now also U2.4
- net MIDI_IN_DATA: now also U2.1
- net MIDI_IN_REF_R: now also U2.3
- net MIDI_UART_RX: now also U2.5
- net USB_DM renamed USB_D_N
- net USB_DM_R renamed USB_DR_N
- net USB_DP renamed USB_D_P
- net USB_DP_R renamed USB_DR_P
Changed lines of the file:
@@
 $Descr A4 11693 8268
 encoding utf-8
-Sheet 3 4
+Sheet 3 5
 Title ""
 Date ""
@@
 F 0 "J6" H 2007 5067 50  0000 C CNN
 F 1 "USB_B_Micro" H 2007 4976 50  0000 C CNN
-F 2 "" H 2100 4550 50  0001 C CNN
+F 2 "Connector_USB:USB_Micro-B_Molex_47346-0001" H 2100 4550 50  0001 C CNN
 F 3 "~" H 2100 4550 50  0001 C CNN
 	1    1950 4600
@@
 F 0 "U3" H 9150 2500 50  0000 C CNN
 F 1 "74LVC1G97" H 9200 2400 50  0000 C CNN
-F 2 "" H 8900 2200 50  0001 C CNN
+F 2 "Package_TO_SOT_SMD:SOT-23-6" H 8900 2200 50  0001 C CNN
 F 3 "http://www.ti.com/lit/sg/scyt129e/scyt129e.pdf" H 8900 2200 50  0001 C CNN
 	1    8900 2200
@@
 $EndComp
 $Comp
-L Isolator:4N35 U2
-U 1 1 5DC748FB
-P 5800 2200
-F 0 "U2" H 5800 2525 50  0000 C CNN
-F 1 "FODM8071" H 5800 2434 50  0000 C CNN
-F 2 "Package_DIP:DIP-6_W7.62mm" H 5600 2000 50  0001 L CIN
-F 3 "https://www.vishay.com/docs/81181/4n35.pdf" H 5800 2200 50  0001 L CNN
-	1    5800 2200
-	1    0    0    -1
-$EndComp
-$Comp
 L Device:D D3
 U 1 1 5DC7644E
 P 4450 2200
 F 0 "D3" V 4404 2279 50  0000 L CNN
-F 1 "D" V 4495 2279 50  0000 L CNN
-F 2 "" H 4450 2200 50  0001 C CNN
+F 1 "1N4148WS" V 4495 2279 50  0000 L CNN
+F 2 "Diode_SMD:D_SOD-323_HandSoldering" H 4450 2200 50  0001 C CNN
 F 3 "~" H 4450 2200 50  0001 C CNN
 	1    4450 2200
@@
 F 0 "R10" V 3895 2400 50  0000 C CNN
 F 1 "220" V 3986 2400 50  0000 C CNN
-F 2 "" V 4140 2390 50  0001 C CNN
+F 2 "Resistor_SMD:R_0603_1608Metric_Pad1.05x0.95mm_HandSolder" V 4140 2390 50  0001 C CNN
 F 3 "~" H 4100 2400 50  0001 C CNN
 	1    4100 2400
@@
 Wire Wire Line
 	5250 2400 5250 2300
-Wire Wire Line
-	5250 2300 5500 2300
 Connection ~ 4450 2400
 Wire Wire Line
@@
 F 0 "J5" H 2822 2124 50  0000 R CNN
 F 1 "Conn_01x02_Male" H 2822 2033 50  0000 R CNN
-F 2 "" H 2850 2150 50  0001 C CNN
+F 2 "Connector_PinHeader_2.54mm:PinHeader_1x02_P2.54mm_Vertical" H 2850 2150 50  0001 C CNN
 F 3 "~" H 2850 2150 50  0001 C CNN
 	1    2850 2150
@@
 F 0 "R11" H 8568 2546 50  0000 L CNN
 F 1 "10k" H 8568 2455 50  0000 L CNN
-F 2 "" V 8540 2490 50  0001 C CNN
+F 2 "Resistor_SMD:R_0603_1608Metric_Pad1.05x0.95mm_HandSolder" V 8540 2490 50  0001 C CNN
 F 3 "~" H 8500 2500 50  0001 C CNN
 	1    8500 2500
@@
 F 0 "R13" V 3945 4600 50  0000 C CNN
 F 1 "27" V 4036 4600 50  0000 C CNN
-F 2 "" V 4190 4590 50  0001 C CNN
+F 2 "Resistor_SMD:R_0603_1608Metric_Pad1.05x0.95mm_HandSolder" V 4190 4590 50  0001 C CNN
 F 3 "~" H 4150 4600 50  0001 C CNN
 	1    4150 4600
@@
 F 0 "R14" V 4263 4700 50  0000 C CNN
 F 1 "27" V 4354 4700 50  0000 C CNN
-F 2 "" V 4190 4690 50  0001 C CNN
+F 2 "Resistor_SMD:R_0603_1608Metric_Pad1.05x0.95mm_HandSolder" V 4190 4690 50  0001 C CNN
 F 3 "~" H 4150 4700 50  0001 C CNN
 	1    4150 4700
@@
 	2700 4600 3800 4600
 Text Label 2950 4600 0    50   ~ 0
-USB_DM
+USB_D_N
 Text Label 2950 4700 0    50   ~ 0
-USB_DP
+USB_D_P
 Text Label 4600 4600 0    50   ~ 0
-USB_DM_R
+USB_DR_N
 Text Label 4600 4700 0    50   ~ 0
-USB_DP_R
+USB_DR_P
 $Comp
 L Device:C C13
@@
 F 0 "C13" H 3915 5046 50  0000 L CNN
 F 1 "47pF" H 3915 4955 50  0000 L CNN
-F 2 "" H 3838 4850 50  0001 C CNN
+F 2 "Capacitor_SMD:C_0603_1608Metric_Pad1.05x0.95mm_HandSolder" H 3838 4850 50  0001 C CNN
 F 3 "~" H 3800 5000 50  0001 C CNN
 	1    3800 5000
@@
 F 0 "C12" H 3386 5046 50  0000 R CNN
 F 1 "47pF" H 3386 4955 50  0000 R CNN
-F 2 "" H 3538 4850 50  0001 C CNN
+F 2 "Capacitor_SMD:C_0603_1608Metric_Pad1.05x0.95mm_HandSolder" H 3538 4850 50  0001 C CNN
 F 3 "~" H 3500 5000 50  0001 C CNN
 	1    3500 5000
@@
 F 0 "C11" H 2865 4146 50  0000 L CNN
 F 1 "0.01uF" H 2865 4055 50  0000 L CNN
-F 2 "" H 2788 3950 50  0001 C CNN
+F 2 "Capacitor_SMD:C_0603_1608Metric_Pad1.05x0.95mm_HandSolder" H 2788 3950 50  0001 C CNN
 F 3 "~" H 2750 4100 50  0001 C CNN
 	1    2750 4100
@@
 F 0 "C9" H 6965 3796 50  0000 L CNN
 F 1 "4.7uF" H 6965 3705 50  0000 L CNN
-F 2 "" H 6888 3600 50  0001 C CNN
+F 2 "Capacitor_SMD:C_0603_1608Metric_Pad1.05x0.95mm_HandSolder" H 6888 3600 50  0001 C CNN
 F 3 "~" H 6850 3750 50  0001 C CNN
 	1    6850 3750
@@
 F 0 "R12" H 4432 4196 50  0000 R CNN
 F 1 "10k" H 4432 4105 50  0000 R CNN
-F 2 "" V 4540 4140 50  0001 C CNN
+F 2 "Resistor_SMD:R_0603_1608Metric_Pad1.05x0.95mm_HandSolder" V 4540 4140 50  0001 C CNN
 F 3 "~" H 4500 4150 50  0001 C CNN
 	1    4500 4150
@@
 F 0 "C8" H 6486 3796 50  0000 R CNN
 F 1 "0.1uF" H 6486 3705 50  0000 R CNN
-F 2 "" H 6638 3600 50  0001 C CNN
+F 2 "Capacitor_SMD:C_0603_1608Metric_Pad1.05x0.95mm_HandSolder" H 6638 3600 50  0001 C CNN
 F 3 "~" H 6600 3750 50  0001 C CNN
 	1    6600 3750
@@
 F 0 "C10" H 4736 3946 50  0000 R CNN
 F 1 "0.1uF" H 4736 3855 50  0000 R CNN
-F 2 "" H 4888 3750 50  0001 C CNN
+F 2 "Capacitor_SMD:C_0603_1608Metric_Pad1.05x0.95mm_HandSolder" H 4888 3750 50  0001 C CNN
 F 3 "~" H 4850 3900 50  0001 C CNN
 	1    4850 3900
@@
 F 0 "D4" H 8643 4995 50  0000 C CNN
 F 1 "LED" H 8643 5086 50  0000 C CNN
-F 2 "" H 8650 5250 50  0001 C CNN
+F 2 "LED_SMD:LED_0805_2012Metric_Pad1.15x1.40mm_HandSolder" H 8650 5250 50  0001 C CNN
 F 3 "~" H 8650 5250 50  0001 C CNN
 	1    8650 5250
@@
 F 0 "D5" H 8643 5573 50  0000 C CNN
 F 1 "LED" H 8643 5664 50  0000 C CNN
-F 2 "" H 8650 5450 50  0001 C CNN
+F 2 "LED_SMD:LED_0805_2012Metric_Pad1.15x1.40mm_HandSolder" H 8650 5450 50  0001 C CNN
 F 3 "~" H 8650 5450 50  0001 C CNN
 	1    8650 5450
@@
 F 0 "R15" V 7595 5250 50  0000 C CNN
 F 1 "220" V 7686 5250 50  0000 C CNN
-F 2 "" V 7840 5240 50  0001 C CNN
+F 2 "Resistor_SMD:R_0603_1608Metric_Pad1.05x0.95mm_HandSolder" V 7840 5240 50  0001 C CNN
 F 3 "~" H 7800 5250 50  0001 C CNN
 	1    7800 5250
@@
 F 0 "R16" V 7913 5450 50  0000 C CNN
 F 1 "220" V 8004 5450 50  0000 C CNN
-F 2 "" V 7840 5440 50  0001 C CNN
+F 2 "Resistor_SMD:R_0603_1608Metric_Pad1.05x0.95mm_HandSolder" V 7840 5440 50  0001 C CNN
 F 3 "~" H 7800 5450 50  0001 C CNN
 	1    7800 5450
@@
 	6850 4800 6850 4900
 NoConn ~ 6550 4700
+$Comp
+L wiproc-rescue:FODM8071-fodm8071 U?
+U 1 1 5DB57638
+P 5800 2200
+AR Path="/5DB57638" Ref="U?"  Part="1"
+AR Path="/5DC68A7B/5DB57638" Ref="U2"  Part="1"
+F 0 "U2" H 5800 2525 50  0000 C CNN
+F 1 "FODM8071" H 5800 2434 50  0000 C CNN
+F 2 "Package_SO:SO-5_4.4x3.6mm_P1.27mm" H 5600 2000 50  0001 L CIN
+F 3 "https://www.vishay.com/docs/83725/4n25.pdf" H 5800 2200 50  0001 L CNN
+	1    5800 2200
+	1    0    0    -1
+$EndComp
+Wire Wire Line
+	5250 2300 5500 2300
 $EndSCHEMATC
