File: pcb/wiproc/wiproc/wiproc.sch (KiCad schematic (older format))
At the start: 10 parts

Commit message: first cut of wiproc schematic
Parts:
- removed C? (x2): C, symbol Device:C
- removed J?: Conn_02x03_Odd_Even, symbol Connector_Generic:Conn_02x03_Odd_Even
- removed J?: USB_B_Micro, symbol Connector:USB_B_Micro
- removed J?: DIN-5, symbol Connector:DIN-5
- removed U?: ATmega328P-AU, Package_QFP:TQFP-32_7x7mm_P0.8mm, symbol MCU_Microchip_ATmega:ATmega328P-AU
- removed U?: FT231XS, Package_SO:SSOP-20_3.9x8.7mm_P0.635mm, symbol Interface_USB:FT231XS
- removed U? (x2): 74LVC1G97, symbol 74xGxx:74LVC1G97
- removed Y?: Crystal, symbol Device:Crystal
- added C1: 0.1uF, symbol Device:C
- added J1: Conn_01x10_Female, symbol Connector:Conn_01x10_Female
- added J2: Conn_01x10_Female_xbee, symbol conn_01x10_female_xbee:Conn_01x10_Female_xbee
- added J3: Conn_02x07_Odd_Even, symbol Connector_Generic:Conn_02x07_Odd_Even
Connections:
- net labels added: +3V3, ADC_IN1, ADC_IN2, I2C_SCL, I2C_SDA, SPARE_IO_1, SPARE_IO_2, XBEE_DOUT, XBEE_RST_N, XPI_SS_N
- net labels removed: +3.3V, +5V, SPI_SS_N, XTAL1_16MHZ, XTAL2_16MHZ
- wire segments 45 -> 86
- no-connect marks 0 -> 11
Other:
- note added: "NOTE:\nDo not populate battery \ncharging manager and \nregulator for synthesizer\nprocessing board."

Commit message: routed wiproc, created synth pcb
Parts:
- C1: footprint (none) -> Capacitor_SMD:C_0603_1608Metric_Pad1.05x0.95mm_HandSolder
- J1, J2: footprint (none) -> Connector_PinSocket_2.00mm:PinSocket_1x10_P2.00mm_Vertical
- J3: footprint (none) -> Connector_PinHeader_2.54mm:PinHeader_2x07_P2.54mm_Vertical
Connections:
- net ADC_IN1: no longer J3.11 (Pin_11)
- net ADC_IN2: no longer J3.12 (Pin_12)
- new net AN_IN1: J3.12 (Pin_12)
- new net AN_IN2: J3.11 (Pin_11)
Other:
- moved on the sheet: C1, J1, J2, J3
