File: pcb/synth/synth/mux.sch (KiCad schematic (older format))
At the start: 3 parts

Commit message: analog synth updates
Parts:
- added C19, C20, C21, C22, C25, C26, C27, C28: 0.1u, Capacitor_SMD:C_0603_1608Metric_Pad1.05x0.95mm_HandSolder, symbol Device:C
- added C24: 1uF, Capacitor_SMD:C_0603_1608Metric_Pad1.05x0.95mm_HandSolder, symbol Device:C
- added J4, J5: Conn_01x02, Connector_PinHeader_2.54mm:PinHeader_1x02_P2.54mm_Vertical, symbol Connector_Generic:Conn_01x02
- added R31: 50, Resistor_SMD:R_0603_1608Metric_Pad1.05x0.95mm_HandSolder, symbol Device:R_US
- added TP1, TP2, TP3, TP4, TP5, TP6: TestPoint, TestPoint:TestPoint_Pad_2.0x2.0mm, symbol Connector:TestPoint
- added U10: OPA172IDBVR, Package_TO_SOT_SMD:SOT-23-5, symbol opa172idbvr:OPA172IDBVR
- added U11, U9: MUX508, Package_SO:SOIC-16_3.9x9.9mm_P1.27mm, symbol mux508:MUX508
- C23: renamed from C?; footprint (none) -> Capacitor_SMD:C_0603_1608Metric_Pad1.05x0.95mm_HandSolder
- R30: renamed from R?; footprint (none) -> Resistor_SMD:R_0603_1608Metric_Pad1.05x0.95mm_HandSolder
- gave numbers to parts that had none: 1
Connections:
- net labels added: AN_BPF, AN_HPF, AN_LPF, AN_SIN, AN_SQR, AN_TRI, FLT_MUX_A0, FLT_MUX_A1, FLT_MUX_A2, FLT_MUX_EN, FLT_MUX_OUT, GND, WF_MUX_A0, WF_MUX_A1, WF_MUX_A2, WF_MUX_EN, WF_MUX_OUT
- net labels removed: MUX_OUT
- wire segments 11 -> 115
Other:
- moved on the sheet: C23, R30, U8

Commit message: final pcb designs and initial i2c
Parts:
- BPF1: renamed from TP5; footprint TestPoint:TestPoint_Pad_2.0x2.0mm -> TestPoint:TestPoint_Pad_1.0x1.0mm
- HPF1: renamed from TP6; footprint TestPoint:TestPoint_Pad_2.0x2.0mm -> TestPoint:TestPoint_Pad_1.0x1.0mm
- LPF1: renamed from TP4; footprint TestPoint:TestPoint_Pad_2.0x2.0mm -> TestPoint:TestPoint_Pad_1.0x1.0mm
- SIN1: renamed from TP1; footprint TestPoint:TestPoint_Pad_2.0x2.0mm -> TestPoint:TestPoint_Pad_1.0x1.0mm
- SQR1: renamed from TP2; footprint TestPoint:TestPoint_Pad_2.0x2.0mm -> TestPoint:TestPoint_Pad_1.0x1.0mm
- TRI1: renamed from TP3; footprint TestPoint:TestPoint_Pad_2.0x2.0mm -> TestPoint:TestPoint_Pad_1.0x1.0mm
Changed lines of the file:
@@
 	5400 3100 5400 3000
 $Comp
-L Connector:TestPoint TP1
+L Connector:TestPoint SIN1
 U 1 1 5DBFF314
 P 4650 2450
-F 0 "TP1" H 4708 2522 50  0000 L CNN
+F 0 "SIN1" H 4708 2522 50  0000 L CNN
 F 1 "TestPoint" H 4708 2477 50  0001 L CNN
-F 2 "TestPoint:TestPoint_Pad_2.0x2.0mm" H 4850 2450 50  0001 C CNN
+F 2 "TestPoint:TestPoint_Pad_1.0x1.0mm" H 4850 2450 50  0001 C CNN
 F 3 "~" H 4850 2450 50  0001 C CNN
 	1    4650 2450
@@
 $EndComp
 $Comp
-L Connector:TestPoint TP2
+L Connector:TestPoint SQR1
 U 1 1 5DC00F70
 P 4900 2450
-F 0 "TP2" H 4958 2522 50  0000 L CNN
+F 0 "SQR1" H 4958 2522 50  0000 L CNN
 F 1 "TestPoint" H 4958 2477 50  0001 L CNN
-F 2 "TestPoint:TestPoint_Pad_2.0x2.0mm" H 5100 2450 50  0001 C CNN
+F 2 "TestPoint:TestPoint_Pad_1.0x1.0mm" H 5100 2450 50  0001 C CNN
 F 3 "~" H 5100 2450 50  0001 C CNN
 	1    4900 2450
@@
 $EndComp
 $Comp
-L Connector:TestPoint TP3
+L Connector:TestPoint TRI1
 U 1 1 5DC015E9
 P 5150 2450
-F 0 "TP3" H 5208 2522 50  0000 L CNN
+F 0 "TRI1" H 5208 2522 50  0000 L CNN
 F 1 "TestPoint" H 5208 2477 50  0001 L CNN
-F 2 "TestPoint:TestPoint_Pad_2.0x2.0mm" H 5350 2450 50  0001 C CNN
+F 2 "TestPoint:TestPoint_Pad_1.0x1.0mm" H 5350 2450 50  0001 C CNN
 F 3 "~" H 5350 2450 50  0001 C CNN
 	1    5150 2450
@@
 	5400 5600 5400 5500
 $Comp
-L Connector:TestPoint TP5
+L Connector:TestPoint BPF1
 U 1 1 5DC0B3A9
 P 4900 4950
-F 0 "TP5" H 4958 5022 50  0000 L CNN
+F 0 "BPF1" H 4958 5022 50  0000 L CNN
 F 1 "TestPoint" H 4958 4977 50  0001 L CNN
-F 2 "TestPoint:TestPoint_Pad_2.0x2.0mm" H 5100 4950 50  0001 C CNN
+F 2 "TestPoint:TestPoint_Pad_1.0x1.0mm" H 5100 4950 50  0001 C CNN
 F 3 "~" H 5100 4950 50  0001 C CNN
 	1    4900 4950
@@
 $EndComp
 $Comp
-L Connector:TestPoint TP6
+L Connector:TestPoint HPF1
 U 1 1 5DC0B3B3
 P 5150 4950
-F 0 "TP6" H 5208 5022 50  0000 L CNN
+F 0 "HPF1" H 5208 5022 50  0000 L CNN
 F 1 "TestPoint" H 5208 4977 50  0001 L CNN
-F 2 "TestPoint:TestPoint_Pad_2.0x2.0mm" H 5350 4950 50  0001 C CNN
+F 2 "TestPoint:TestPoint_Pad_1.0x1.0mm" H 5350 4950 50  0001 C CNN
 F 3 "~" H 5350 4950 50  0001 C CNN
 	1    5150 4950
@@
 	5400 4900 5400 5500
 $Comp
-L Connector:TestPoint TP4
+L Connector:TestPoint LPF1
 U 1 1 5DC270B5
 P 4650 4950
-F 0 "TP4" H 4708 5022 50  0000 L CNN
+F 0 "LPF1" H 4708 5022 50  0000 L CNN
 F 1 "TestPoint" H 4708 4977 50  0001 L CNN
-F 2 "TestPoint:TestPoint_Pad_2.0x2.0mm" H 4850 4950 50  0001 C CNN
+F 2 "TestPoint:TestPoint_Pad_1.0x1.0mm" H 4850 4950 50  0001 C CNN
 F 3 "~" H 4850 4950 50  0001 C CNN
 	1    4650 4950
