File: pcb/synth/synth/synth.kicad_pcb (KiCad board)
At the start: 2 copper layers, 116 parts, among them J1 Screw_Terminal_01x06, J2 AudioJack2, J3 Conn_02x07_Odd_Even, J4 Conn_01x02, J5 Conn_01x02, U1 LM13700, U10 OPA172IDBVR, U11 MUX508, U12 PCF8574A, U13 AD5694R, U14 LM386, U2 LM13700, U3 LM13700, U4 LM13700, U5 LM13700, U6 OPA172IDBVR, U7 OPA172IDBVR, U8 OPA172IDBVR, U9 MUX508

Commit message: inital synth schematic
Parts:
- added C39: 0.1u, Capacitor_SMD:C_0603_1608Metric_Pad1.05x0.95mm_HandSolder, F.Cu at (231.8, 123.2)
- added C40: 0.1u, Capacitor_SMD:C_0603_1608Metric_Pad1.05x0.95mm_HandSolder, F.Cu at (231.8, 130.7)
- added C41: 0.1u, Capacitor_SMD:C_0603_1608Metric_Pad1.05x0.95mm_HandSolder, F.Cu at (231.8, 146.4)
- added C42: 0.1u, Capacitor_SMD:C_0603_1608Metric_Pad1.05x0.95mm_HandSolder, F.Cu at (240.5, 138.9)
- added C43: 0.1u, Capacitor_SMD:C_0603_1608Metric_Pad1.05x0.95mm_HandSolder, F.Cu at (243.4, 107.3)
- added C44: 0.1u, Capacitor_SMD:C_0603_1608Metric_Pad1.05x0.95mm_HandSolder, F.Cu at (243.4, 104.8)
- added C45: 1u, Capacitor_SMD:C_0603_1608Metric_Pad1.05x0.95mm_HandSolder, F.Cu at (204.5, 137.2)
- added C46: 0.1u, Capacitor_SMD:C_0603_1608Metric_Pad1.05x0.95mm_HandSolder, F.Cu at (204.5, 139.7)
- added C47: 10u, Capacitor_SMD:C_0603_1608Metric_Pad1.05x0.95mm_HandSolder, F.Cu at (208.8, 137.2)
- added C48: 0.1u, Capacitor_SMD:C_0603_1608Metric_Pad1.05x0.95mm_HandSolder, F.Cu at (204.5, 142.2)
- added C49: 0.1u, Capacitor_SMD:C_0603_1608Metric_Pad1.05x0.95mm_HandSolder, F.Cu at (208.8, 139.7)
- added R54: 10k, Resistor_SMD:R_0603_1608Metric_Pad1.05x0.95mm_HandSolder, F.Cu at (240.5, 123.2)
- added R55: 10k, Resistor_SMD:R_0603_1608Metric_Pad1.05x0.95mm_HandSolder, F.Cu at (236.1, 125.7)
- added R56: 10k, Resistor_SMD:R_0603_1608Metric_Pad1.05x0.95mm_HandSolder, F.Cu at (231.8, 120.7)
- added R57: 10k, Resistor_SMD:R_0603_1608Metric_Pad1.05x0.95mm_HandSolder, F.Cu at (231.8, 128.2)
- added R58: 1.2k, Resistor_SMD:R_0603_1608Metric_Pad1.05x0.95mm_HandSolder, F.Cu at (240.5, 120.7)
- added R59: 10k, Resistor_SMD:R_0603_1608Metric_Pad1.05x0.95mm_HandSolder, F.Cu at (236.1, 123.2)
- added R60: 10k, Resistor_SMD:R_0603_1608Metric_Pad1.05x0.95mm_HandSolder, F.Cu at (231.8, 125.7)
- added R61: 10k, Resistor_SMD:R_0603_1608Metric_Pad1.05x0.95mm_HandSolder, F.Cu at (236.1, 120.7)
- added R62: 10k, Resistor_SMD:R_0603_1608Metric_Pad1.05x0.95mm_HandSolder, F.Cu at (236.1, 141.4)
- added R63: 10k, Resistor_SMD:R_0603_1608Metric_Pad1.05x0.95mm_HandSolder, F.Cu at (231.8, 143.9)
- added R64: 10k, Resistor_SMD:R_0603_1608Metric_Pad1.05x0.95mm_HandSolder, F.Cu at (231.8, 136.4)
- added R65: 10k, Resistor_SMD:R_0603_1608Metric_Pad1.05x0.95mm_HandSolder, F.Cu at (240.5, 136.4)
- added R66: 1.2k, Resistor_SMD:R_0603_1608Metric_Pad1.05x0.95mm_HandSolder, F.Cu at (236.1, 138.9)
- added R67: 10k, Resistor_SMD:R_0603_1608Metric_Pad1.05x0.95mm_HandSolder, F.Cu at (231.8, 141.4)
- added R68: 10k, Resistor_SMD:R_0603_1608Metric_Pad1.05x0.95mm_HandSolder, F.Cu at (231.8, 138.9)
- added R69: 10k, Resistor_SMD:R_0603_1608Metric_Pad1.05x0.95mm_HandSolder, F.Cu at (236.1, 136.4)
- added R70: 10k, Resistor_SMD:R_0603_1608Metric_Pad1.05x0.95mm_HandSolder, F.Cu at (247.7, 104.8)
- added R71: 10k, Resistor_SMD:R_0603_1608Metric_Pad1.05x0.95mm_HandSolder, F.Cu at (243.4, 109.8)
- added R72: 10k, Resistor_SMD:R_0603_1608Metric_Pad1.05x0.95mm_HandSolder, F.Cu at (247.7, 107.3)
- added R73: 10k, Resistor_SMD:R_0603_1608Metric_Pad1.05x0.95mm_HandSolder, F.Cu at (252.1, 104.8)
- added R74: 1.2k, Resistor_SMD:R_0603_1608Metric_Pad1.05x0.95mm_HandSolder, F.Cu at (243.4, 112.3)
- added R75: 10k, Resistor_SMD:R_0603_1608Metric_Pad1.05x0.95mm_HandSolder, F.Cu at (247.7, 109.8)
- added R76: 10k, Resistor_SMD:R_0603_1608Metric_Pad1.05x0.95mm_HandSolder, F.Cu at (252.1, 107.3)
- added R77: 10k, Resistor_SMD:R_0603_1608Metric_Pad1.05x0.95mm_HandSolder, F.Cu at (243.4, 114.8)
- added R78: 10k, Resistor_SMD:R_0603_1608Metric_Pad1.05x0.95mm_HandSolder, F.Cu at (213.2, 137.2)
- added R79: 10k, Resistor_SMD:R_0603_1608Metric_Pad1.05x0.95mm_HandSolder, F.Cu at (204.5, 144.7)
- added R80: 10k, Resistor_SMD:R_0603_1608Metric_Pad1.05x0.95mm_HandSolder, F.Cu at (208.8, 142.2)
- added R81: 10k, Resistor_SMD:R_0603_1608Metric_Pad1.05x0.95mm_HandSolder, F.Cu at (213.2, 139.7)
- added R82: 10k, Resistor_SMD:R_0603_1608Metric_Pad1.05x0.95mm_HandSolder, F.Cu at (217.5, 137.2)
- added U14: OPA4172, Package_SO:SOIC-14_3.9x8.7mm_P1.27mm, F.Cu at (225.4, 124.5)
- added U15: OPA4172, Package_SO:SOIC-14_3.9x8.7mm_P1.27mm, F.Cu at (225.4, 140.2)
- added U16: OPA4172, Package_SO:SOIC-14_3.9x8.7mm_P1.27mm, F.Cu at (237.0, 108.7)
Connections:
- net /mux/FLT_MUX_A2 renamed /dig_ctrl/FLT_MUX_A2
- net Net-(U12-Pad6) renamed /dig_ctrl/WF_MUX_A1
- net Net-(U12-Pad7) renamed /dig_ctrl/WF_MUX_A2
- U11 pad 1: /mux/FLT_MUX_A0 -> /dig_ctrl/FLT_MUX_A0
- U11 pad 16: /mux/FLT_MUX_A1 -> /dig_ctrl/FLT_MUX_A1
- U11 pad 2: /mux/FLT_MUX_EN -> /dig_ctrl/FLT_MUX_EN
- U12 pad 1: Net-(U12-Pad1) -> GND
- U12 pad 10: Net-(U12-Pad10) -> /dig_ctrl/FLT_MUX_A0
- U12 pad 11: Net-(U12-Pad11) -> /dig_ctrl/FLT_MUX_A1
- U12 pad 14: Net-(U12-Pad14) -> /I2C_SCL
- U12 pad 15: Net-(U12-Pad15) -> /I2C_SDA
- U12 pad 16: Net-(U12-Pad16) -> +3V3
- U12 pad 2: Net-(U12-Pad2) -> GND
- U12 pad 3: Net-(U12-Pad3) -> GND
- U12 pad 8: Net-(U12-Pad8) -> GND
- U12 pad 9: Net-(U12-Pad9) -> /dig_ctrl/FLT_MUX_EN
- U13 pad 10: Net-(U13-Pad10) -> GND
- U13 pad 11: Net-(U13-Pad11) -> +3V3
- U13 pad 12: Net-(U13-Pad12) -> GND
- U13 pad 13: Net-(U13-Pad13) -> /I2C_SCL
- U13 pad 14: Net-(U13-Pad14) -> GND
- U13 pad 2: Net-(U13-Pad2) -> /dig_ctrl/ana_scale_vcf/AN_IN
- U13 pad 3: Net-(U13-Pad3) -> /dig_ctrl/ana_scale_vco/AN_IN
- U13 pad 4: Net-(U13-Pad4) -> GND
- U13 pad 5: Net-(U13-Pad5) -> +3V3
- U13 pad 6: Net-(U13-Pad6) -> /dig_ctrl/ana_scale_vca/AN_IN
- U13 pad 8: Net-(U13-Pad8) -> /I2C_SDA
- U13 pad 9: Net-(U13-Pad9) -> /SPARE_IO_2

Commit message: final pcb designs and initial i2c
Parts:
- removed the U14 at (226.1, 113.4)
- added C51: 10u, Capacitor_SMD:C_0603_1608Metric_Pad1.05x0.95mm_HandSolder, B.Cu at (210.6, 106.4)
- added C52: 10u, Capacitor_SMD:C_0603_1608Metric_Pad1.05x0.95mm_HandSolder, B.Cu at (208.8, 83.2)
- added C53: 10u, Capacitor_SMD:C_0603_1608Metric_Pad1.05x0.95mm_HandSolder, B.Cu at (210.6, 116.7)
- added REF**: MountingHole_3.5mm_Pad, MountingHole:MountingHole_3.5mm_Pad, F.Cu at (146.1, 128.3)
- added REF**: MountingHole_3.5mm_Pad, MountingHole:MountingHole_3.5mm_Pad, F.Cu at (146.1, 85.1)
- added REF**: MountingHole_3.5mm_Pad, MountingHole:MountingHole_3.5mm_Pad, F.Cu at (214.6, 128.3)
- added REF**: MountingHole_3.5mm_Pad, MountingHole:MountingHole_3.5mm_Pad, F.Cu at (214.6, 85.1)
- added TP1: TestPoint, TestPoint:TestPoint_Pad_1.0x1.0mm, B.Cu at (187.2, 85.7)
- added TP10: TestPoint, TestPoint:TestPoint_Pad_1.0x1.0mm, B.Cu at (187.7, 98.3)
- added TP2: TestPoint, TestPoint:TestPoint_Pad_1.0x1.0mm, B.Cu at (208.0, 85.3)
- added TP3: TestPoint, TestPoint:TestPoint_Pad_1.0x1.0mm, B.Cu at (187.2, 83.2)
- BPF1: renamed from TP5; footprint TestPoint:TestPoint_Pad_2.0x2.0mm -> TestPoint:TestPoint_Pad_1.0x1.0mm
- C12, C18, C34, C37, C39, C40, C41, C42, C43, C44, C45, C46, C47, C48, C49, R54, R55, R56, R57, R58, R59, R60, R61, R62, R63, R64, R65, R66, R67, R68, R69, R70, R71, R72, R73, R74, R75, R76, R77, R78, R79, R80, U13, U14, U15, U16: moved to B.Cu
- HPF1: renamed from TP6; footprint TestPoint:TestPoint_Pad_2.0x2.0mm -> TestPoint:TestPoint_Pad_1.0x1.0mm
- LPF1: renamed from TP4; footprint TestPoint:TestPoint_Pad_2.0x2.0mm -> TestPoint:TestPoint_Pad_1.0x1.0mm
- R50: value 47k -> 51k
- R81, R82: value 10k -> 1.2k; moved to B.Cu
- SIN1: renamed from TP1; footprint TestPoint:TestPoint_Pad_2.0x2.0mm -> TestPoint:TestPoint_Pad_1.0x1.0mm
- SQR1: renamed from TP2; footprint TestPoint:TestPoint_Pad_2.0x2.0mm -> TestPoint:TestPoint_Pad_1.0x1.0mm
- TRI1: renamed from TP3; footprint TestPoint:TestPoint_Pad_2.0x2.0mm -> TestPoint:TestPoint_Pad_1.0x1.0mm
- U12: footprint Package_SO:SOIC-16W-12_7.5x10.3mm_P1.27mm -> Package_SO:SOIC-16W_7.5x10.3mm_P1.27mm; moved to B.Cu
- moved R58 79.8 mm to (160.8, 124.9), turned to 270 degrees
- moved R57 74.4 mm to (158.0, 119.0), turned to 90 degrees
- moved J1 73.0 mm to (214.0, 94.0), turned to 270 degrees
- moved R60 72.0 mm to (160.8, 113.5), turned to 180 degrees
- moved R54 70.8 mm to (169.7, 122.4), turned to 90 degrees
- moved R55 70.8 mm to (166.5, 113.1), turned to 270 degrees
- moved C40 70.1 mm to (163.9, 113.1), turned to 270 degrees
- moved R65 69.8 mm to (172.9, 118.9), turned to 90 degrees
- moved R56 69.2 mm to (162.7, 124.9), turned to 90 degrees
- moved C37 68.6 mm to (148.0, 100.3), turned to 90 degrees
- moved C39 67.2 mm to (164.6, 124.9), turned to 270 degrees
- moved C42 66.8 mm to (179.0, 113.0), turned to 270 degrees
- moved R61 66.7 mm to (169.7, 115.3), turned to 270 degrees
- moved R59 66.6 mm to (169.7, 118.8), turned to 90 degrees
- moved R73 65.3 mm to (188.5, 119.4), turned to 90 degrees
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Connections:
- J1 pad 1: -12V -> +3V3
- J1 pad 5: +3V3 -> -12V
- J3 pad 1: /MCU_RST_N -> +3V3
- J3 pad 2: +3V3 -> /MCU_RST_N
- J3 pad 5: /I2C_SCL -> /SPARE_IO_1
- J3 pad 6: /SPARE_IO_1 -> /I2C_SCL
- J3 pad 7: /I2C_SDA -> /SPARE_IO_2
- J3 pad 8: /SPARE_IO_2 -> /I2C_SDA
- U9 pad 1: /mux/WF_MUX_A0 -> /dig_ctrl/WF_MUX_A0
- U9 pad 15: /mux/WF_MUX_A2 -> /dig_ctrl/WF_MUX_A2
- U9 pad 16: /mux/WF_MUX_A1 -> /dig_ctrl/WF_MUX_A1
- U9 pad 2: /mux/WF_MUX_EN -> /dig_ctrl/WF_MUX_EN
Routing:
- net GND: track 0.00 -> 168.0 mm, vias 0 -> 57
- net -12V: track 0.00 -> 92.3 mm, vias 0 -> 22
- net +12V: track 0.00 -> 71.6 mm, vias 0 -> 18
- net /mux/AN_SIN: track 0.00 -> 64.1 mm, vias 0 -> 3
- net /vcf/AN_VCF_IN: track 0.00 -> 57.0 mm, vias 0 -> 4
- net /mux/AN_SQR: track 0.00 -> 54.2 mm
- net /mux/AN_HPF: track 0.00 -> 49.0 mm, vias 0 -> 2
- net /dig_ctrl/ana_scale_vco/AN_IN: track 0.00 -> 48.1 mm
- net /dig_ctrl/WF_MUX_A0: track 0.00 -> 46.7 mm, vias 0 -> 1
- net /dig_ctrl/WF_MUX_EN: track 0.00 -> 45.9 mm, vias 0 -> 1
- net /dig_ctrl/CTRL_VCO: track 0.00 -> 44.4 mm, vias 0 -> 3
- net /mux/AN_TRI: track 0.00 -> 44.2 mm
- net Net-(R37-Pad2): track 0.00 -> 36.6 mm
- net /mux/AN_BPF: track 0.00 -> 34.3 mm, vias 0 -> 2
- net /dig_ctrl/WF_MUX_A2: track 0.00 -> 32.6 mm, vias 0 -> 1
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- added copper zone on In2.Cu, net +12V
- added copper zone on In2.Cu, net +3V3
- added copper zone on B.Cu, net -12V
- added copper zone on In1.Cu, net GND
Other:
- board outline added: 76.2 x 50.8 mm
- copper layers 2 -> 4
- net class Default: clearance 0.2 -> 0.2032; trace_width 0.25 -> 0.254; via_dia 0.8 -> 0.762; via_drill 0.4 -> 0.381
- net class Power added: clearance 0.254, trace_width 0.381, via_dia 0.762, via_drill 0.381
- rule pad_to_mask_clearance: 0.051 -> 0.0508
- rule solder_mask_min_width: 0.25 -> 0.1016
- rule trace_clearance: 0.2 -> 0.2032
- rule trace_min: 0.2 -> 0.1524
- rule via_min_drill: 0.3 -> 0.254
- rule via_min_size: 0.4 -> 0.508
- board text added: "ANALOG"
- board text added: "SYNTHESIZER"
- board text added: "V1.0"
