File: pcb/synth/synth/synth.sch (KiCad schematic (older format))
At the start: 0 parts

Commit message: analog synth updates
Parts:
- added J1: Screw_Terminal_01x06, TerminalBlock:TerminalBlock_bornier-6_P5.08mm, symbol Connector:Screw_Terminal_01x06
- added J2: AudioJack2, Connector_PinHeader_2.54mm:PinHeader_1x02_P2.54mm_Vertical, symbol Connector:AudioJack2
- added J3: Conn_02x07_Odd_Even, Connector_PinHeader_2.54mm:PinHeader_2x07_P2.54mm_Vertical, symbol Connector_Generic:Conn_02x07_Odd_Even
Connections:
- net labels added: +12V, +3V3, -12V, AN_1, AN_2, GND, I2C_SCL, I2C_SDA, MCU_RST_N, SPARE_IO_1, SPARE_IO_2
- wire segments 0 -> 64

Commit message: inital synth schematic
Connections:
- wire segments 64 -> 81
Other:
- moved on the sheet: J1, J2, J3

Commit message: final pcb designs and initial i2c
Parts:
- added C51, C52, C53: 10u, Capacitor_SMD:C_0603_1608Metric_Pad1.05x0.95mm_HandSolder, symbol Device:C
- added TP1, TP2, TP3: TestPoint, TestPoint:TestPoint_Pad_1.0x1.0mm, symbol Connector:TestPoint
Connections:
- wire segments 81 -> 93
Other:
- moved on the sheet: J1, J2, J3
