File: pcb/synth/synth/vca.sch (KiCad schematic (older format))
At the start: 9 parts, among them U5 LM13700

Commit message: final pcb designs and initial i2c
Parts:
- R50: value 47k -> 51k
Changed lines of the file:
@@
 P 6600 4000
 F 0 "R50" H 6532 3954 50  0000 R CNN
-F 1 "47k" H 6532 4045 50  0000 R CNN
+F 1 "51k" H 6532 4045 50  0000 R CNN
 F 2 "Resistor_SMD:R_0603_1608Metric_Pad1.05x0.95mm_HandSolder" V 6640 3990 50  0001 C CNN
 F 3 "~" H 6600 4000 50  0001 C CNN
