File: pcb/synth/synth/vcf.sch (KiCad schematic (older format))
At the start: 26 parts, among them U4 LM13700, U5 LM13700

Commit message: final pcb designs and initial i2c
Connections:
- no-connect marks 0 -> 3
Changed lines of the file:
@@
 Wire Wire Line
 	4000 6700 4000 6750
+NoConn ~ 6450 2550
+NoConn ~ 4200 5050
+NoConn ~ 4100 2550
 $EndSCHEMATC
